File: hw/4-20ma-mcu.kicad_pcb (KiCad board)
At the start: 2 copper layers, 39 parts, among them J2 Conn_01x04_Male, U1 L7805, U2 LM324A, U3 ATtiny84A-SS, U4 74AHC1G04, Y1 16MHz 20pF

Commit message: dev update 030725=1
Parts:
- added C14: 10uF, Capacitor_SMD:C_1206_3216Metric, F.Cu at (123.0, 86.8)
- added R14: 15K, Resistor_SMD:R_0805_2012Metric, F.Cu at (115.6, 90.8)
- C10: value 0.1uF -> 1uF
- C13: value 10uF -> 0.1uF
- C3: footprint Capacitor_SMD:C_0805_2012Metric -> Capacitor_SMD:C_1206_3216Metric
- C7: value 10pF -> 0.1uF; footprint Capacitor_SMD:C_0603_1608Metric -> Capacitor_SMD:C_0805_2012Metric
- C9: value 1uF -> 10pF; footprint Capacitor_SMD:C_0805_2012Metric -> Capacitor_SMD:C_0603_1608Metric
- R10: value 100R -> 10K
- R11: value 21K -> 100R
- R12: value 4.75K -> 21K
- R13: value 15K -> 4.75K
- R2, R6: value 10K -> 1K
- R4: value 1K -> 10K
- moved U1 71.4 mm to (110.0, 60.1), turned to 90 degrees
- moved C7 44.8 mm to (115.5, 77.0)
- moved D3 40.2 mm to (115.3, 94.0), turned to 180 degrees
- moved Y1 35.0 mm to (137.8, 65.5)
- moved C3 34.2 mm to (108.0, 68.8), turned to -90 degrees
- moved C2 29.0 mm to (110.5, 68.3), turned to -90 degrees
- moved C13 27.7 mm to (108.5, 93.0), turned to 180 degrees
- moved U2 27.6 mm to (115.5, 83.0)
- moved U4 26.9 mm to (129.4, 83.8), turned to 180 degrees
- moved D1 26.3 mm to (121.8, 73.0)
- moved F1 25.1 mm to (123.5, 66.1), turned to -90 degrees
- moved C10 22.8 mm to (108.6, 88.0), turned to 180 degrees
- moved R12 21.8 mm to (115.6, 88.8)
- moved J2 21.7 mm to (137.4, 94.8), turned to 90 degrees
- moved R6 20.9 mm to (143.0, 72.8)
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Connections:
- C10 pad 1: Net-(U3-~{RESET}/PB3) -> Net-(C10-Pad1)
- C10 pad 2: GND -> Net-(U2B--)
- C11 pad 1: GND -> Net-(U3-~{RESET}/PB3)
- C11 pad 2: +5V -> GND
- C12 pad 1: Net-(D3-A) -> GND
- C12 pad 2: GND -> +5V
- C13 pad 1: Net-(U2C-+) -> Net-(D3-A)
- C4 pad 1: Net-(U2D-+) -> V_IN
- C5 pad 1: GND -> Net-(U2D-+)
- C5 pad 2: +5V -> GND
- C6 pad 1: +5V -> GND
- C6 pad 2: GND -> +5V
- C7 pad 1: Net-(U3-XTAL1/PB0) -> +5V
- C8 pad 1: Net-(U3-XTAL2/PB1) -> Net-(U3-XTAL1/PB0)
- C9 pad 1: Net-(C9-Pad1) -> Net-(U3-XTAL2/PB1)
- C9 pad 2: Net-(U2B--) -> GND
- R10 pad 1: Net-(D3-A) -> Net-(U3-~{RESET}/PB3)
- R10 pad 2: Net-(C9-Pad1) -> +5V
- R11 pad 1: Net-(U2B-+) -> Net-(D3-A)
- R11 pad 2: Net-(U2C--) -> Net-(C10-Pad1)
- R12 pad 1: Net-(U2C-+) -> Net-(U2B-+)
- R12 pad 2: Net-(R12-Pad2) -> Net-(U2C--)
- R13 pad 1: GND -> Net-(U2C-+)
- R13 pad 2: Net-(U2B-+) -> Net-(R13-Pad2)
- R2 pad 1: Net-(U2A--) -> Net-(U2D--)
- R2 pad 2: Net-(R2-Pad2) -> V_IN
- R3 pad 1: Net-(D3-A) -> Net-(U2A--)
- R3 pad 2: Net-(U2A--) -> Net-(R3-Pad2)
- R4 pad 1: Net-(R4-Pad1) -> Net-(D3-A)
- R4 pad 2: +5V -> Net-(U2A--)
- R5 pad 1: GND -> Net-(R5-Pad1)
- R5 pad 2: Net-(R5-Pad2) -> +5V
- R6 pad 1: Net-(U2B--) -> GND
- R6 pad 2: Net-(R2-Pad2) -> Net-(R6-Pad2)
- R7 pad 1: Net-(U2A-+) -> Net-(U2B--)
- R7 pad 2: GND -> Net-(R3-Pad2)
- R8 pad 1: Net-(C9-Pad1) -> Net-(U2A-+)
- R8 pad 2: Net-(U2A-+) -> GND
- R9 pad 1: Net-(U3-~{RESET}/PB3) -> Net-(C10-Pad1)
- R9 pad 2: +5V -> Net-(U2A-+)
- RV1 pad 1: Net-(R4-Pad1) -> Net-(R5-Pad1)
- RV1 pad 3: Net-(R5-Pad2) -> Net-(R6-Pad2)
- U2 pad 1: Net-(R2-Pad2) -> Net-(R3-Pad2)
- U2 pad 13: V_IN -> Net-(U2D--)
- U2 pad 14: V_IN -> Net-(U2D--)
- U2 pad 7: Net-(C9-Pad1) -> Net-(C10-Pad1)
- U4 pad 4: Net-(R12-Pad2) -> Net-(R13-Pad2)
