File: hw/4-20ma-mcu.kicad_sch (KiCad schematic)
At the start: 4 parts, among them U1 ATtiny84A-SS, U2 LM324A

Commit message: dev update 030425
Parts:
- removed unit 4 of U2
- added C2: 10uF, Capacitor_SMD:C_1206_3216Metric, symbol Device:C_Polarized
- added C3, C4, C5, C6, C7: 0.1uF, Capacitor_SMD:C_0805_2012Metric, symbol Device:C
- added D1: D_Schottky, Package_TO_SOT_SMD:SOT-23, symbol Device:D_Schottky
- added R10: 4.75K, R_0805_2012Metric, symbol Device:R
- added R2, R3, R4, R5, R6: 10K, R_0805_2012Metric, symbol Device:R
- added R7: 100R, R_0805_2012Metric, symbol Device:R
- added R8: 21K, R_0805_2012Metric, symbol Device:R
- added R9: 15K, R_0805_2012Metric, symbol Device:R
- added U3: 74AHC1G04, Package_TO_SOT_SMD:SOT-23-5, symbol 74xGxx:74AHC1G04
- C1: value 100nF -> 1uF; footprint C_0805_2012Metric_Pad1.18x1.45mm_HandSolder -> Capacitor_SMD:C_0805_2012Metric
Connections:
- net +5V: now also R1.2, U1.1 (VCC), U2.4 (V+), C3.1, C4.2, C5.2, U3.5 (VCC)
- net GND: now also U1.14 (GND), U2.11 (V-), C2.2, C3.2, C4.1, C5.1, C6.2, C7.2, R4.2, R9.1, U3.3 (GND)
- net at U2.1: now also R2.2, R6.2
- net at U2.2 (-): now also R2.1, R3.2
- net at U2.3 (+): now also R4.1, R5.2
- net at U2.5 (+): now also R8.1, R9.2
- net at U2.6 (-): now also C1.2, R6.1
- net at U2.7: now also C1.1, R5.1, R7.2
- net at U2.10 (+): now also C2.1, R10.1
- net at U2.8: now also U2.9 (-), R8.2
- net at R1.1: now also U1.4 (~{RESET}/PB3), C6.1
- new net: C7.1, D1.2 (A), R3.1, R7.1
- new net: R10.2, U3.4
- new net PWM: U3.2
- new net SIG_OUT: D1.1 (K)
Other:
- note added: "${DateCreated}"
- note added: "${Engineer}"
- note added: "${Revision}"
- note added: "${SheetNum}"
- note added: "${SheetTotal}"
- note added: "${Title}"
- moved on the sheet: C1, R1, U1, U2A, U2B, U2C, U2E

Commit message: 030525
Parts:
- added J1: ~, TerminalBlock_Phoenix:TerminalBlock_Phoenix_MKDS-1,5-4-5.08_1x04_P5.08mm_Horizontal, symbol lib-030525:Term_Block_4p_5.08mm
Connections:
- net PWM: now also U1.7 (PA6)
- net A_IN: now reaches U1.13 (AREF/PA0)
Changed lines of the file:
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@@
+	(wire
+		(pts
+			(xy 80.01 59.69) (xy 83.82 59.69)
+		)
+		(stroke
+			(width 0)
+			(type default)
+		)
+	)
 	(wire
 		(pts
@@
 	(wire
 		(pts
+			(xy 80.01 74.93) (xy 83.82 74.93)
+		)
+		(stroke
+			(width 0)
+			(type default)
+		)
+	)
+	(wire
+		(pts
 			(xy 138.43 125.73) (xy 138.43 129.54)
 		)
@@
 			(width 0)
 			(type default)
+		)
+	)
+	(global_label "A_IN"
+		(shape input)
+		(at 83.82 59.69 0)
+		(fields_autoplaced yes)
+		(effects
+			(font
+				(size 1.27 1.27)
+			)
+			(justify left)
+		)
+		(property "Intersheetrefs" "${INTERSHEET_REFS}"
+			(at 90.7967 59.69 0)
+			(effects
+				(font
+					(size 1.27 1.27)
+				)
+				(justify left)
+				(hide yes)
+			)
 		)
 	)
@@
 				)
 				(justify right)
+				(hide yes)
+			)
+		)
+	)
+	(global_label "PWM"
+		(shape output)
+		(at 83.82 74.93 0)
+		(fields_autoplaced yes)
+		(effects
+			(font
+				(size 1.27 1.27)
+			)
+			(justify left)
+		)
+		(property "Intersheetrefs" "${INTERSHEET_REFS}"
+			(at 90.978 74.93 0)
+			(effects
+				(font
+					(size 1.27 1.27)
+				)
+				(justify left)
 				(hide yes)
 			)
@@
 					(unit 1)
 				)
+			)
+		)
+	)
+	(symbol
+		(lib_id "lib-030525:Term_Block_4p_5.08mm")
+		(at 260.35 33.02 0)
+		(unit 1)
+		(exclude_from_sim no)
+		(in_bom yes)
+		(on_board yes)
+		(dnp no)
+		(fields_autoplaced yes)
+		(property "Reference" "J1"
+			(at 264.16 32.3849 0)
+			(effects
+				(font
+					(size 1.27 1.27)
+				)
+				(justify left)
+			)
+		)
+		(property "Value" "~"
+			(at 264.16 34.29 0)
+			(effects
+				(font
+					(size 1.27 1.27)
+				)
+				(justify left)
+			)
+		)
+		(property "Footprint" "TerminalBlock_Phoenix:TerminalBlock_Phoenix_MKDS-1,5-4-5.08_1x04_P5.08mm_Horizontal"
+			(at 260.35 33.02 0)
+			(effects
+				(font
+					(size 1.27 1.27)
+				)
+				(hide yes)
+			)
+		)
+		(property "Datasheet" ""
+			(at 260.35 33.02 0)
+			(effects
+				(font
+					(size 1.27 1.27)
+				)
+				(hide yes)
+			)
+		)
+		(property "Description" "Weidmuller 1146380000"
+			(at 260.35 33.02 0)
+			(effects
+				(font
+					(size 1.27 1.27)
+				)
+				(hide yes)
+			)
+		)
+		(pin "3"
+		)
+		(pin "2"
+		)
+		(pin "1"
+		)
+		(pin "4"
+		)
+		(instances
+			(project ""
+				(path "/3ebdbe86-dc72-4c13-868e-7208cc88469e"
+					(reference "J1")
+					(unit 1)
+				)

Commit message: dev update 030525-1
Parts:
- removed C2: 10uF, Capacitor_SMD:C_1206_3216Metric, symbol Device:C_Polarized
- added C10, C11: 10uF, Capacitor_SMD:C_0805_2012Metric, symbol Device:C
- added C12, C9: 0.1uF, Capacitor_SMD:C_0805_2012Metric, symbol Device:C
- added C8: 0.33uF, Capacitor_SMD:C_0805_2012Metric, symbol Device:C
- added D2: SCHOTTKY 30V 1A, Package_TO_SOT_SMD:SOT-23, symbol Device:D_Schottky
- added D3: TVS 30V 600W, Diode_SMD:D_SMB, symbol tvs-diode:TVS_Diode_Uni
- added F1: PTC FUSE 30V 0.5 A, Fuse:Fuse_1812_4532Metric, symbol Device:Polyfuse
- added FB1: 150 ohm @ 100 MHz 4LN, Resistor_SMD:R_0805_2012Metric, symbol Device:FerriteBead_Small
- added J2: Conn_01x04_Male, Connector_PinHeader_2.54mm:PinHeader_1x04_P2.54mm_Vertical, symbol Connector:Conn_01x04_Male
- added R11: 1K, R_0805_2012Metric, symbol Device:R
- added U4: L7805, Package_TO_SOT_SMD:TO-252-2, symbol Regulator_Linear:L7805
- D1: value D_Schottky -> SCHOTTKY 70V 200mW
Connections:
- net SIG_OUT is gone; now on net mA_OUT: D1.1 (K)
- net +5V: now also C11.1, C9.1, J2.1 (Pin_1), U4.3 (OUT)
- net GND: now also J1.4, C10.2, C11.2, C12.2, C8.2, C9.2, D3., J2.4 (Pin_4), U4.2 (GND)
- net at R10.1, U2.10 (+): now also C10.1
- net DC_IN: now reaches J1.1
- net DC_IN: now also F1.1
- net at J1.2: now also FB1.2
- net mA_OUT: now reaches J1.3
- net TX: now reaches U1.6 (PA7)
- net TX: now also J2.3 (Pin_3)
- net A_IN renamed V_IN
- net V_IN: now also U2.13 (-), U2.14
- new net: C8.1, D2.1 (K), D3., U4.1 (IN)
- new net: C12.1, R11.2, U2.12 (+)
- new net: FB1.1, R11.1
- new net: D2.2 (A), F1.2
- new net RX: J2.2 (Pin_2)
Other:
- moved on the sheet: C3, C5, C6, D1, J1, R1, U1, U2E

Commit message: dev update 030625-0
Parts:
- added C13, C2: 6pF, Capacitor_SMD:C_0603_1608Metric, symbol Device:C_Small
- added RV1: 4.7K, Potentiometer_SMD:Potentiometer_Bourns_TC33X_Vertical, symbol Device:R_Potentiometer_Trim
- added unit 4 of U2
- added Y1: 16MHz 20pF, Crystal:Crystal_SMD_HC49-SD, symbol Device:Crystal
Connections:
- net GND: now also C13.2, C2.2
- net TX: now also U1.8 (PA5); no longer U1.6 (PA7)
- net V_IN: now also U2.13 (-), U2.14; no longer U2.13 (-), U2.14
- net at C12.1, R11.2: now also U2.12 (+); no longer U2.12 (+)
- net at U1.2 (XTAL1/PB0): now also C2.1, Y1.2
- net at U1.3 (XTAL2/PB1): now also C13.1, Y1.1
- net RX renamed RX_NC
Other:
- moved on the sheet: C6

Commit message: dev update 030725-0
Parts:
- added R4, R5: 1K, R_0805_2012Metric, symbol Device:R
- C7: renamed from C2; value 6pF -> 10pF
- C8: renamed from C13; value 6pF -> 10pF
- D1: renamed from D2; footprint Package_TO_SOT_SMD:SOT-23 -> Diode_SMD:D_SMB
- D3: renamed from D1; footprint Package_TO_SOT_SMD:SOT-23 -> Diode_SMD:D_SMB
- renumbered C8 to C1, C6 to C10, C4 to C11, C7 to C12, C10 to C13, C9 to C2, C11 to C3, C12 to C4, C3 to C6, C1 to C9, D3 to D2, R11 to R1, R7 to R10, R8 to R11, R10 to R12, R9 to R13, R4 to R7, R5 to R8, R1 to R9, U4 to U1, U1 to U3, U3 to U4
Connections:
- net +5V: now also R4.2
- net GND: now also D2.2, R5.1; no longer D2.
- net at C1.1, D1.1 (K), U1.1 (IN): now also D2.1; no longer D2.
- net at RV1.1: now also R4.1
- net at RV1.2: now also U3.12 (PA1)
- net at RV1.3: now also R5.2
Other:
- note added: "mA TRIM"
- moved on the sheet: C10, C11, C12, C13, C5, C6, C7, C8, C9, D3, R10, R11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

Commit message: dev update 030725=1
Parts:
- added C4: 0.1uF, Capacitor_SMD:C_0805_2012Metric, symbol Device:C
- added R2: 1K, R_0805_2012Metric, symbol Device:R
- C14: renamed from C13; footprint Capacitor_SMD:C_0805_2012Metric -> Capacitor_SMD:C_1206_3216Metric
- C3: footprint Capacitor_SMD:C_0805_2012Metric -> Capacitor_SMD:C_1206_3216Metric
- renumbered C9 to C10, C10 to C11, C11 to C12, C12 to C13, C4 to C5, C5 to C6, C6 to C7, C7 to C8, C8 to C9, R9 to R10, R10 to R11, R11 to R12, R12 to R13, R13 to R14, R2 to R3, R3 to R4, R4 to R5, R5 to R6, R6 to R7, R7 to R8, R8 to R9
Connections:
- net GND: now also C4.2
- net V_IN: now also C4.1, R2.2; no longer U2.13 (-), U2.14
- new net: R2.1, U2.13 (-), U2.14
